Commit message: geometry done

File: ball_shooter_sim/urdf/ball_shooter.xacro (robot description, xacro)
@@ -26,10 +26,15 @@
 <!--***************************Pluguins***************************-->
 <!--***************************Variables***************************-->
-<xacro:property name="base_link_length" value="0.1" />
+<xacro:property name="base_link_length" value="0.02" />
 <xacro:property name="base_link_radius" value="0.2" />
-<xacro:property name="pan_link_length" value="0.1" />
+<xacro:property name="pan_link_length" value="0.02" />
 <xacro:property name="pan_link_radius" value="0.2" />
+<xacro:property name="camera_link_height" value="0.2" />
+<xacro:property name="camera_link_width" value="0.2" />
+<xacro:property name="camera_link_hegth" value="0.01" />
 <xacro:property name="tilt_link_length" value="0.4" />
 <xacro:property name="tilt_link_radius" value="0.04" />
+<xacro:property name="ball_suport_height" value="0.03" />
+<xacro:property name="ball_suport_width" value="0.06" />
 <!--***************************Variables***************************-->
 <!--***************************Links***************************-->
@@ -78,4 +83,29 @@
   </inertial>
 </link>
+<!-- Support ball -->
+<!-- <link name="ball_support_link">
+  <origin xyz="0 0 ${ball_suport_height/2}" rpy="0 0 0" />
+  <visual>
+    <origin xyz="0 0 ${ball_suport_height/2}" rpy="0 0 0" />
+    <geometry>
+      <box size="${ball_suport_width} ${ball_suport_width} ${ball_suport_height}"/>
+    </geometry>
+    <material name="blue"/>
+  </visual>
+  <collision>
+    <origin xyz="0 0 ${ball_suport_height/2}" rpy="0 0 0" />
+    <geometry>
+      <box size="${ball_suport_width} ${ball_suport_width} ${ball_suport_height}"/>
+    </geometry>
+  </collision>
+  <inertial>
+    <origin xyz="0 0 ${ball_suport_height/2}" rpy="0 0 0" />
+    <mass value="0.1"/>
+  <inertia
+    ixx="0.00041666666666666675" ixy="0.0" ixz="0.0"
+    iyy="0.00041666666666666675" iyz="0.0"
+    izz="0.000166667"/>
+    </inertial>
+</link> -->
 <!-- camera_link -->
 <link name="camera_link">
@@ -112,5 +142,5 @@
   <parent link="base_link"/>
   <child link="pan_link"/>
-  <origin xyz="0 0 0.1"/>
+  <origin xyz="0 0 0.025"/>
   <axis xyz="0 0 1" />
   <limit effort="300" velocity="1" lower="-3.14" upper="3.14"/>
@@ -121,7 +151,14 @@
   <parent link="pan_link"/>
   <child link="camera_link"/>
-  <origin rpy="0 0 0" xyz="0.0 0.0 0.06"/>
+  <origin rpy="0 0 0" xyz="0.055 0.0 0.015"/>
   <axis xyz="0 0 0" />
 </joint>
+<!-- ball_suport_link -->
+<!-- <joint name="ball_support_joint" type="fixed">
+  <parent link="pan_link"/>
+  <child link="ball_support_link"/>
+  <origin rpy="0 0 0" xyz="0.2 0 0.015"/>
+  <axis xyz="0 0 0" />
+</joint> -->
 <!-- dummy_camera_joint -->
 <joint name="dummy_camera_joint" type="fixed">

Commit message: ball_shooter ball ok

File: ball_shooter_sim/urdf/ball_shooter.xacro (robot description, xacro)
@@ -27,7 +27,7 @@
 <!--***************************Variables***************************-->
 <xacro:property name="base_link_length" value="0.02" />
-<xacro:property name="base_link_radius" value="0.2" />
+<xacro:property name="base_link_radius" value="0.1" />
 <xacro:property name="pan_link_length" value="0.02" />
-<xacro:property name="pan_link_radius" value="0.2" />
+<xacro:property name="pan_link_radius" value="0.1" />
 <xacro:property name="camera_link_height" value="0.2" />
 <xacro:property name="camera_link_width" value="0.2" />
@@ -35,8 +35,9 @@
 <xacro:property name="tilt_link_length" value="0.4" />
 <xacro:property name="tilt_link_radius" value="0.04" />
-<xacro:property name="ball_suport_height" value="0.03" />
-<xacro:property name="ball_suport_width" value="0.06" />
+<xacro:property name="ball_suport_height" value="0.035" />
+<xacro:property name="ball_suport_width" value="0.05" />
 <!--***************************Variables***************************-->
 <!--***************************Links***************************-->
+<!-- <link name="world" /> -->
 <!-- base_link -->
 <link name="base_link">
@@ -52,5 +53,5 @@
   <collision>
     <geometry>
-      <cylinder length="${base_link_length+0.02}" radius="${base_link_radius}"/>
+      <cylinder length="${base_link_length}" radius="${base_link_radius}"/>
     </geometry>
     <origin rpy="0 0 0" xyz="0 0 0"/>
@@ -67,5 +68,5 @@
       <cylinder length="${pan_link_length}" radius="${pan_link_radius}"/>
     </geometry>
-    <origin rpy="0 0 0" xyz="0 0 0."/>
+    <origin rpy="0 0 0" xyz="0 0 0"/>
     <material name="blue">
       <color rgba="0 0 1 1"/>
@@ -74,7 +75,7 @@
   <collision>
     <geometry>
-      <cylinder length="${pan_link_length}" radius="${pan_link_radius+0.02}"/>
-    </geometry>
-    <origin rpy="0 0 0" xyz="0 0 0.09"/>
+      <cylinder length="${pan_link_length}" radius="${pan_link_radius}"/>
+    </geometry>
+    <origin rpy="0 0 0" xyz="0 0 0.0"/>
   </collision>
   <inertial>
@@ -84,5 +85,5 @@
 </link>
 <!-- Support ball -->
-<!-- <link name="ball_support_link">
+<link name="ball_support_link">
   <origin xyz="0 0 ${ball_suport_height/2}" rpy="0 0 0" />
   <visual>
@@ -107,24 +108,24 @@
     izz="0.000166667"/>
     </inertial>
-</link> -->
+</link>
 <!-- camera_link -->
-<link name="camera_link">
-  <origin xyz="0 0 0.05" rpy="0 0 0" />
-  <visual>
-    <origin xyz="0 0 0.05" rpy="0 0 0" />
-    <geometry>
-      <box size="0.1 0.1 0.1"/>
+<!-- <link name="camera_link">
+  <origin xyz="0 0 0.025" rpy="0 0 0" />
+  <visual>
+    <origin xyz="0 0 0.025" rpy="0 0 0" />
+    <geometry>
+      <box size="0.05 0.05 0.05"/>
     </geometry>
     <material name="blue"/>
   </visual>
   <collision>
-    <origin xyz="0 0 0.05" rpy="0 0 0" />
-    <geometry>
-      <box size="0.1 0.1 0.1"/>
-    </geometry>
-  </collision>
-  <inertial>
-    <origin xyz="0 0 0.05" rpy="0 0 0" />
-    <mass value="0.1"/>
+    <origin xyz="0 0 0.025" rpy="0 0 0" />
+    <geometry>
+      <box size="0.05 0.05 0.05"/>
+    </geometry>
+  </collision>
+  <inertial>
+    <origin xyz="0 0 0.025" rpy="0 0 0" />
+    <mass value="0"/>
   <inertia
     ixx="0.000166667" ixy="0.0" ixz="0.0"
@@ -132,10 +133,15 @@
     izz="0.000166667"/>
     </inertial>
-</link>
+</link> -->
 <!-- dummy_camera_link -->
-<link name="dummy_camera_link">
-</link>
+<!-- <link name="dummy_camera_link">
+</link> -->
 <!--***************************Links***************************-->
 <!--***************************Joints***************************-->
+<!-- <joint name="world_to_base_link=" type="fixed">
+     <parent link="world"/>
+     <child link="base_link"/>
+    <origin xyz="0 0 0.01"/>
+</joint> -->
 <!-- pan_joint -->
 <joint name="pan_joint" type="revolute">
@@ -148,24 +154,30 @@
 </joint>
 <!-- camera_joint -->
-<joint name="camera_joint" type="fixed">
+<!-- <joint name="camera_joint" type="fixed">
   <parent link="pan_link"/>
   <child link="camera_link"/>
   <origin rpy="0 0 0" xyz="0.055 0.0 0.015"/>
   <axis xyz="0 0 0" />
-</joint>
+</joint> -->
+<!-- <joint name="camera_joint" type="fixed">
+  <parent link="base_link"/>
+  <child link="camera_link"/>
+  <origin rpy="0 0 0" xyz="0.135 0.0 0.015"/>
+  <axis xyz="0 0 0" />
+</joint> -->
 <!-- ball_suport_link -->
-<!-- <joint name="ball_support_joint" type="fixed">
+<joint name="ball_support_joint" type="fixed">
   <parent link="pan_link"/>
   <child link="ball_support_link"/>
-  <origin rpy="0 0 0" xyz="0.2 0 0.015"/>
-  <axis xyz="0 0 0" />
-</joint> -->
+  <origin rpy="0 0 0" xyz="0.06 0 0.015"/>
+  <axis xyz="0 0 0" />
+</joint>
 <!-- dummy_camera_joint -->
-<joint name="dummy_camera_joint" type="fixed">
+<!-- <joint name="dummy_camera_joint" type="fixed">
   <parent link="camera_link"/>
   <child link="dummy_camera_link"/>
-  <origin rpy="0 0 0" xyz="0 0 0.05"/>
-  <axis xyz="0 0 0" />
-</joint>
+  <origin rpy="0 0 0" xyz="0 0 0.025"/>
+  <axis xyz="0 0 0" />
+</joint> -->
 <!--***************************Joints***************************-->
 <!--***************************Gazebo configuration***************************-->
@@ -173,5 +185,4 @@
 <gazebo reference="base_link">
   <material>Gazebo/Red</material>
-  <turnGravityOff>True</turnGravityOff>
 </gazebo>
 <!-- pan_link -->
@@ -180,10 +191,9 @@
 </gazebo>
 <!-- dummy_camera_link -->
-<gazebo reference="dummy_camera_link">
+<!-- <gazebo reference="dummy_camera_link">
   <sensor type="camera" name="camera1">
     <update_rate>30</update_rate>
     <always_on>1</always_on>
     <visualize>true</visualize>
-  <!-- <pose>0 0 0.05 0 0 0</pose> -->
   <camera name="head">
     <horizontal_fov>1.047</horizontal_fov>
@@ -205,7 +215,4 @@
     <cameraInfoTopicName>camera_info</cameraInfoTopicName>
     <frameName>camera_link_optical</frameName>
-    <!-- setting hackBaseline to anything but 0.0 will cause a misalignment
-      between the gazebo sensor image and the frame it is supposed to
-      be attached to -->
     <hackBaseline>0.0</hackBaseline>
     <distortionK1>0.0</distortionK1>
@@ -220,5 +227,5 @@
   </plugin>
   </sensor>
-</gazebo>
+</gazebo> -->
 <!--***************************Gazebo configuration***************************-->
 <!--***************************Transmissions***************************-->
